Commit message: Attach Robotiq 2F-85 gripper to UR5e via ur_to_robotiq adapter
- Chain: tool0 -> ur_to_robotiq adapter -> robotiq_gripper -> tcp_link
- tcp_link added as functional grasp frame (measured fingertip depth
  0.098m via tf2_echo)
- Manual ros2_control block for the gripper (include_ros2_control=false
  on the macro) since the packaged robotiq_description macro gives every
  mimic joint its own command_interface, which ros2_control's resource
  manager rejects outright

File: ros2_ws/src/robot_control_pkg/urdf/ur_positioned.urdf.xacro (robot description, xacro)
@@ -22,3 +22,42 @@
     <origin xyz="0.8 -0.45 0.70" rpy="0 0 1.5708" />
   </xacro:ur_robot>
+  <!-- ================= Robotiq 2F-85 gripper ================= -->
+  <xacro:include filename="$(find robotiq_description)/urdf/ur_to_robotiq_adapter.urdf.xacro" />
+  <xacro:include filename="$(find robotiq_description)/urdf/robotiq_2f_85_macro.urdf.xacro" />
+  <!-- tool0 -> adapter plate -> gripper_mount_link -->
+  <xacro:ur_to_robotiq
+      prefix=""
+      connected_to="tool0"
+      rotation="0.0" />
+  <!-- gripper_mount_link -> robotiq_85_base_link -> fingers -->
+  <xacro:robotiq_gripper
+      name="RobotiqGripperHardwareInterface"
+      prefix=""
+      parent="gripper_mount_link"
+      use_fake_hardware="true"
+      include_ros2_control="false">
+    <origin xyz="0 0 0" rpy="0 0 0" />
+  </xacro:robotiq_gripper>
+  <!-- Manual ros2_control block: only the real actuated joint gets a command
+       interface. Mimic joints (right knuckle, inner knuckles, finger tips)
+       derive their state from the <mimic> tag in the plain URDF joint below —
+       giving them their own command_interface is what crashed ros2_control_node. -->
+  <ros2_control name="RobotiqGripperHardwareInterface" type="system">
+    <hardware>
+      <plugin>mock_components/GenericSystem</plugin>
+      <param name="state_following_offset">0.0</param>
+    </hardware>
+    <joint name="robotiq_85_left_knuckle_joint">
+      <command_interface name="position"/>
+      <state_interface name="position"/>
+      <state_interface name="velocity"/>
+    </joint>
+  </ros2_control>
+  <!-- Functional grasp/TCP frame: gripper centerline, at measured fingertip depth -->
+  <link name="tcp_link" />
+  <joint name="tcp_joint" type="fixed">
+    <parent link="robotiq_85_base_link" />
+    <child link="tcp_link" />
+    <origin xyz="0 0 0.098" rpy="0 0 0" />
+  </joint>
 </robot>

Commit message: fix base height so it's flush with the table, spawn in home

File: ros2_ws/src/robot_control_pkg/urdf/ur_positioned.urdf.xacro (robot description, xacro)
@@ -20,5 +20,5 @@
     force_abs_paths="false"
     >
-    <origin xyz="0.8 -0.45 0.70" rpy="0 0 1.5708" />
+    <origin xyz="0.8 -0.45 0.752" rpy="0 0 1.5708" />
   </xacro:ur_robot>
   <!-- ================= Robotiq 2F-85 gripper ================= -->

Commit message: add physics-mode bringup: gz_ros2_control, effort-driven gripper, perception launch

File: ros2_ws/src/robot_control_pkg/urdf/ur_positioned.urdf.xacro (robot description, xacro)
@@ -4,4 +4,9 @@
        which hardcodes it and fights our static_transform_publisher node -->
   <xacro:include filename="$(find ur_description)/urdf/ur_macro.xacro" />
+  <!-- true = actuate through Gazebo physics (gz_ros2_control), the arm and
+       gripper actually push against the simulated box instead of MoveIt's
+       planning scene alone deciding what's "attached". false (default) =
+       mock_components/GenericSystem, instant fake actuation, no physics. -->
+  <xacro:arg name="sim_gazebo" default="false" />
   <link name="world" />
   <xacro:ur_robot
@@ -41,13 +46,68 @@
   <ros2_control name="RobotiqGripperHardwareInterface" type="system">
     <hardware>
-      <plugin>mock_components/GenericSystem</plugin>
-      <param name="state_following_offset">0.0</param>
+      <xacro:if value="$(arg sim_gazebo)">
+        <plugin>gz_ros2_control/GazeboSimSystem</plugin>
+      </xacro:if>
+      <xacro:unless value="$(arg sim_gazebo)">
+        <plugin>mock_components/GenericSystem</plugin>
+        <param name="state_following_offset">0.0</param>
+      </xacro:unless>
     </hardware>
     <joint name="robotiq_85_left_knuckle_joint">
-      <command_interface name="position"/>
-      <state_interface name="position"/>
-      <state_interface name="velocity"/>
+      <!-- sim_gazebo: effort command, driven by gripper_effort_controller's
+           closed-loop force logic (command a modest torque and let real
+           contact stop it, instead of driving to a fixed position that a
+           velocity-position servo can't reliably turn into real squeeze
+           force; see gripper_effort_controller.py for why. Position
+           state is still reported for MoveIt/RViz; effort state feeds the
+           stall/contact detection.
+           Fake hardware: unchanged, position-commanded as before. -->
+      <xacro:if value="$(arg sim_gazebo)">
+        <command_interface name="effort"/>
+        <state_interface name="position"/>
+        <state_interface name="velocity"/>
+        <state_interface name="effort"/>
+      </xacro:if>
+      <xacro:unless value="$(arg sim_gazebo)">
+        <command_interface name="position"/>
+        <state_interface name="position"/>
+        <state_interface name="velocity"/>
+      </xacro:unless>
     </joint>
+    <!-- dartsim doesn't enforce the URDF mimic, so the right knuckle hung
+         under gravity; drive it with its own (sign-mirrored) effort. -->
+    <xacro:if value="$(arg sim_gazebo)">
+      <joint name="robotiq_85_right_knuckle_joint">
+        <command_interface name="effort"/>
+        <state_interface name="position"/>
+        <state_interface name="velocity"/>
+        <state_interface name="effort"/>
+      </joint>
+    </xacro:if>
   </ros2_control>
+  <!-- Single gz_ros2_control system plugin for the whole robot: it picks up
+       every <ros2_control> block above (arm's, from ur.ros2_control.xacro,
+       and the gripper's above) under one controller_manager inside Gazebo. -->
+  <xacro:if value="$(arg sim_gazebo)">
+    <gazebo>
+      <plugin filename="gz_ros2_control-system" name="gz_ros2_control::GazeboSimROS2ControlPlugin">
+        <parameters>$(find robot_control_pkg)/config/ros2_controllers.yaml</parameters>
+      </plugin>
+    </gazebo>
+    <!-- Gazebo-native joint spawn angle, independent of ros2_control
+         entirely: without this every arm joint physically spawns at 0
+         (fully extended) regardless of the ros2_control "initial_value"
+         claim, and gz_ros2_control's position-interface servo proved too
+         weak/slow against gravity to actually reach the SRDF "home" pose
+         from there before MoveIt's first plan: it settled partway,
+         drooped enough to intersect the table, and CheckStartStateCollision
+         rejected every plan. Spawning already at home sidesteps needing
+         that servo to do any work at all before the first real trajectory. -->
+    <gazebo reference="shoulder_lift_joint">
+      <axis>
+        <initial_position>-1.5708</initial_position>
+      </axis>
+    </gazebo>
+  </xacro:if>
   <!-- Functional grasp/TCP frame: gripper centerline, at measured fingertip depth -->
   <link name="tcp_link" />

File: ros2_ws/src/ur5e_robotiq_moveit_config/config/ur.ros2_control.xacro (robot description, xacro)
@@ -1,10 +1,29 @@
 <?xml version="1.0"?>
 <robot xmlns:xacro="http://www.ros.org/wiki/xacro">
-    <xacro:macro name="ur_ros2_control" params="name initial_positions_file">
+    <xacro:macro name="ur_ros2_control" params="name initial_positions_file sim_gazebo:=false">
         <xacro:property name="initial_positions" value="${xacro.load_yaml(initial_positions_file)['initial_positions']}"/>
         <ros2_control name="${name}" type="system">
             <hardware>
-                <!-- By default, set up controllers for simulation. This won't work on real hardware -->
-                <plugin>mock_components/GenericSystem</plugin>
+                <!-- sim_gazebo=false (default): mock_components, instant fake
+                     actuation, no physics, won't work on real hardware either.
+                     sim_gazebo=true: actuated through Gazebo physics via the
+                     gz_ros2_control plugin declared in ur_positioned.urdf.xacro. -->
+                <xacro:if value="${sim_gazebo}">
+                    <plugin>gz_ros2_control/GazeboSimSystem</plugin>
+                    <!-- gz_ros2_control's position command interface is a
+                         VELOCITY servo, not a torque PID:
+                         joint_velocity = gain * position_error * update_rate
+                         (100 Hz here). This is a direct child element of
+                         <hardware>, NOT a <param name="..."> (that syntax
+                         is specific to mock_components/GenericSystem):
+                         using <param> here was silently ignored, so every
+                         gain value tried (including absurdly large ones)
+                         produced identical behavior: the plugin was always
+                         falling back to its own default (0.1) regardless. -->
+                    <position_proportional_gain>5.0</position_proportional_gain>
+                </xacro:if>
+                <xacro:unless value="${sim_gazebo}">
+                    <plugin>mock_components/GenericSystem</plugin>
+                </xacro:unless>
             </hardware>
             <joint name="shoulder_pan_joint">

File: ros2_ws/src/ur5e_robotiq_moveit_config/config/ur.urdf.xacro (robot description, xacro)
@@ -2,8 +2,13 @@
 <robot xmlns:xacro="http://www.ros.org/wiki/xacro" name="ur">
     <xacro:arg name="initial_positions_file" default="initial_positions.yaml" />
-    <!-- Import ur urdf file -->
+    <!-- Import ur urdf file. It declares its own sim_gazebo xacro:arg
+         (default false), which is what actually decides mock_components
+         vs gz_ros2_control for the gripper below and (via the macro call
+         below) the arm too. -->
     <xacro:include filename="$(find robot_control_pkg)/urdf/ur_positioned.urdf.xacro" />
     <!-- Import control_xacro -->
     <xacro:include filename="ur.ros2_control.xacro" />
-    <xacro:ur_ros2_control name="FakeSystem" initial_positions_file="$(arg initial_positions_file)"/>
+    <xacro:ur_ros2_control name="UR5eSystem"
+                            initial_positions_file="$(arg initial_positions_file)"
+                            sim_gazebo="$(arg sim_gazebo)"/>
 </robot>
